File: MicroTVbGone_r2.kicad_pcb (KiCad board)
At the start: 16 copper layers, 25.4 x 25.4 mm, 15 parts, among them Q1 2N3904, Q2 2N3904, Q4 2N3904, T1 MMBT2907, U1 ATTINY85V-10SU

Commit message: Reduce stackup to 2 layers and export Gerbers
Other:
- copper layers 16 -> 2
Changed lines of the file:
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@@
 (kicad_pcb (version 20211014) (generator pcbnew)
   (general
-    (thickness 1.6)
+    (thickness 0.158)
   )
   (paper "A4")
   (layers
     (0 "F.Cu" signal)
-    (1 "In1.Cu" signal)
-    (2 "In2.Cu" signal)
-    (3 "In3.Cu" signal)
-    (4 "In4.Cu" signal)
-    (5 "In5.Cu" signal)
-    (6 "In6.Cu" signal)
-    (7 "In7.Cu" signal)
-    (8 "In8.Cu" signal)
-    (9 "In9.Cu" signal)
-    (10 "In10.Cu" signal)
-    (11 "In11.Cu" signal)
-    (12 "In12.Cu" signal)
-    (13 "In13.Cu" signal)
-    (14 "In14.Cu" signal)
     (31 "B.Cu" signal)
     (32 "B.Adhes" user "B.Adhesive")
@@
   )
   (setup
+    (stackup
+      (layer "F.SilkS" (type "Top Silk Screen"))
+      (layer "F.Paste" (type "Top Solder Paste"))
+      (layer "F.Mask" (type "Top Solder Mask") (thickness 0.01))
+      (layer "F.Cu" (type "copper") (thickness 0.035))
+      (layer "dielectric 1" (type "core") (thickness 0.068) (material "FR4") (epsilon_r 4.5) (loss_tangent 0.02))
+      (layer "B.Cu" (type "copper") (thickness 0.035))
+      (layer "B.Mask" (type "Bottom Solder Mask") (thickness 0.01))
+      (layer "B.Paste" (type "Bottom Solder Paste"))
+      (layer "B.SilkS" (type "Bottom Silk Screen"))
+      (copper_finish "None")
+      (dielectric_constraints no)
+    )
     (pad_to_mask_clearance 0)
     (pcbplotparams
